File: MSGEQ7_Breakout_Board/MSGEQ7_Breakout_Board.sch (KiCad schematic (older format))
At the start: 10 parts, among them J1 BREAKOUT_BOARD_HEADER, J2 STEREO_MINI_JACK, U1 MSGEQ7

Commit message: Prototype Layout Completed
Submitted schematic to Mixed Signal Integration and had it validated for
correctness.  Finalized BOM for the prototype and completed layout with
an eye towards producing as a kit: all PTH components, minimum .15"
spacing.
Connections:
- net labels added: GND
- net labels removed: AGND, DGND
- wire segments 33 -> 35
Other:
- note added: "Clarification needed from former backers on \nwhether they prefer stereo mini jack or .1" \nheader for audio input"
- note added: "MSGEQ7 will require 8 pin DIP footprint\nas requested by former backers to aid\nin hand soldering"
- note added: "Six Pin .1" Header"
- moved on the sheet: C1, C2, C3, C4, J2, R1, R2, R3, U1

Commit message: Gerbers and Schematic Completed for Prototype
The layout was modified to accomodate non-oval drills and drill files
were merged.  All manufacturers, part numbers and datasheet fields have
been completed in the schematic.
Parts:
- C1, C2, C4: MFG Name (none) -> Vishay; MFG Part Num (none) -> K103K15X7RF53L2
- C3: MFG Name (none) -> Vishay; MFG Part Num (none) -> K330J15C0GF5TL2
- J1: MFG Name (none) -> Sullins Connector; MFG Part Num (none) -> PREC040SAAN-RC
- J2: MFG Name (none) -> CUI Inc; MFG Part Num (none) -> SJ1-3523NG
- R1: MFG Name (none) -> Stackpole; MFG Part Num (none) -> CF14JT200K
- R2, R3: MFG Name (none) -> Stackpole; MFG Part Num (none) -> CF14JT22K0
- U1: MFG Name (none) -> Mixed Signal Integration; MFG Part Num (none) -> MSGEQ7
Changed lines of the file:
@@
 Sheet 1 1
 Title "MSGEQ7 Breakout Board"
-Date "13 dec 2014"
+Date "7 jan 2015"
 Rev "A"
 Comp "Rheingold Heavy"
@@
 F 1 "MSGEQ7" H 6150 3950 60  0000 C CNN
 F 2 "" H 5900 3950 60  0000 C CNN
-F 3 "" H 5900 3950 60  0000 C CNN
+F 3 "http://www.mix-sig.com/images/datasheets/MSGEQ7.pdf" H 5900 3950 60  0001 C CNN
+F 4 "Mixed Signal Integration" H 6150 3950 60  0001 C CNN "MFG Name"
+F 5 "MSGEQ7" H 6150 3950 60  0001 C CNN "MFG Part Num"
 	1    6150 3950
 	1    0    0    -1
@@
 F 1 "200K" V 6850 3100 40  0000 C CNN
 F 2 "~" V 6780 3100 30  0000 C CNN
-F 3 "~" H 6850 3100 30  0000 C CNN
+F 3 "https://www.seielect.com/catalog/SEI-CF_CFM.pdf" H 6850 3100 30  0001 C CNN
+F 4 "Stackpole" H 6850 3100 60  0001 C CNN "MFG Name"
+F 5 "CF14JT200K" H 6850 3100 60  0001 C CNN "MFG Part Num"
 	1    6850 3100
 	-1   0    0    1
@@
 F 1 "0.1uF" V 5175 3425 40  0000 L CNN
 F 2 "~" H 5338 3350 30  0000 C CNN
-F 3 "~" H 5300 3500 60  0000 C CNN
+F 3 "http://datasheet.octopart.com/K103K15X7RF53L2-Vishay-datasheet-20674387.pdf" H 5300 3500 60  0001 C CNN
+F 4 "Vishay" H 5300 3500 60  0001 C CNN "MFG Name"
+F 5 "K103K15X7RF53L2" H 5300 3500 60  0001 C CNN "MFG Part Num"
 	1    5300 3500
 	0    -1   -1   0
@@
 F 1 "33pF" V 7025 3425 40  0000 L CNN
 F 2 "~" H 7188 3350 30  0000 C CNN
-F 3 "~" H 7150 3500 60  0000 C CNN
+F 3 "http://datasheet.octopart.com/K330J15C0GF5TL2-Vishay-datasheet-13562638.pdf" H 7150 3500 60  0001 C CNN
+F 4 "Vishay" H 7150 3500 60  0001 C CNN "MFG Name"
+F 5 "K330J15C0GF5TL2" H 7150 3500 60  0001 C CNN "MFG Part Num"
 	1    7150 3500
 	0    -1   -1   0
@@
 Text GLabel 5025 4400 0    50   Input ~ 0
 STROBE
-$Comp
-L C C4
-U 1 1 545E8A09
-P 7150 4100
-F 0 "C4" V 7200 3950 40  0000 L CNN
-F 1 "0.1uF" V 7025 4025 40  0000 L CNN
-F 2 "~" H 7188 3950 30  0000 C CNN
-F 3 "~" H 7150 4100 60  0000 C CNN
-	1    7150 4100
-	0    -1   -1   0
-$EndComp
 Wire Wire Line
 	6950 4100 6600 4100
@@
 F 1 "22K" V 7900 4650 40  0000 C CNN
 F 2 "~" V 7830 4650 30  0000 C CNN
-F 3 "~" H 7900 4650 30  0000 C CNN
+F 3 "https://www.seielect.com/catalog/SEI-CF_CFM.pdf" H 7900 4650 30  0001 C CNN
+F 4 "Stackpole" H 7900 4650 60  0001 C CNN "MFG Name"
+F 5 "CF14JT22K0" H 7900 4650 60  0001 C CNN "MFG Part Num"
 	1    7900 4650
-	0    -1   -1   0
-$EndComp
-$Comp
-L R R3
-U 1 1 545E8AC6
-P 7900 4850
-F 0 "R3" V 7980 4850 40  0000 C CNN
-F 1 "22K" V 7900 4850 40  0000 C CNN
-F 2 "~" V 7830 4850 30  0000 C CNN
-F 3 "~" H 7900 4850 30  0000 C CNN
-	1    7900 4850
 	0    -1   -1   0
 $EndComp
@@
 F 1 "BREAKOUT_BOARD_HEADER" V 3000 3950 50  0000 C CNN
 F 2 "" H 3400 4100 60  0000 C CNN
-F 3 "" H 3400 4100 60  0000 C CNN
+F 3 "http://media.digikey.com/PDF/Data%20Sheets/Sullins%20PDFs/z%20RzCzzzSzzN-RC,%20ST,11635-B.pdf" H 3400 4100 60  0001 C CNN
+F 4 "Sullins Connector" H 3250 3950 60  0001 C CNN "MFG Name"
+F 5 "PREC040SAAN-RC" H 3250 3950 60  0001 C CNN "MFG Part Num"
 	1    3250 3950
 	1    0    0    -1
@@
 Wire Wire Line
 	7450 4750 7350 4750
-$Comp
-L C C2
-U 1 1 54669D08
-P 7150 4750
-F 0 "C2" V 7200 4600 40  0000 L CNN
-F 1 "0.1uF" V 7025 4675 40  0000 L CNN
-F 2 "~" H 7188 4600 30  0000 C CNN
-F 3 "~" H 7150 4750 60  0000 C CNN
-	1    7150 4750
-	0    -1   -1   0
-$EndComp
 Wire Wire Line
 	6750 4750 6950 4750
@@
 F 1 "STEREO_MINI_JACK" H 8650 5200 60  0000 C CNN
 F 2 "" H 8750 4850 60  0000 C CNN
-F 3 "" H 8750 4850 60  0000 C CNN
+F 3 "http://www.cui.com/product/resource/sj1-352xng-series.pdf" H 8750 4850 60  0001 C CNN
+F 4 "CUI Inc" H 8650 4850 60  0001 C CNN "MFG Name"
+F 5 "SJ1-3523NG" H 8650 4850 60  0001 C CNN "MFG Part Num"
 	1    8650 4850
 	1    0    0    -1
@@
 Wire Notes Line
 	8600 5300 8600 5650
+$Comp
+L C C2
+U 1 1 54AD6E03
+P 7150 4750
+F 0 "C2" V 7200 4600 40  0000 L CNN
+F 1 "0.1uF" V 7025 4675 40  0000 L CNN
+F 2 "~" H 7188 4600 30  0000 C CNN
+F 3 "http://datasheet.octopart.com/K103K15X7RF53L2-Vishay-datasheet-20674387.pdf" H 7150 4750 60  0001 C CNN
+F 4 "Vishay" H 7150 4750 60  0001 C CNN "MFG Name"
+F 5 "K103K15X7RF53L2" H 7150 4750 60  0001 C CNN "MFG Part Num"
+	1    7150 4750
+	0    -1   -1   0
+$EndComp
+$Comp
+L C C4
+U 1 1 54AD6E2B
+P 7150 4100
+F 0 "C4" V 7200 3950 40  0000 L CNN
+F 1 "0.1uF" V 7025 4025 40  0000 L CNN
+F 2 "~" H 7188 3950 30  0000 C CNN
+F 3 "http://datasheet.octopart.com/K103K15X7RF53L2-Vishay-datasheet-20674387.pdf" H 7150 4100 60  0001 C CNN
+F 4 "Vishay" H 7150 4100 60  0001 C CNN "MFG Name"
+F 5 "K103K15X7RF53L2" H 7150 4100 60  0001 C CNN "MFG Part Num"
+	1    7150 4100
+	0    -1   -1   0
+$EndComp
+$Comp
+L R R3
+U 1 1 54AD6E77
+P 7900 4850
+F 0 "R3" V 7980 4850 40  0000 C CNN
+F 1 "22K" V 7900 4850 40  0000 C CNN
+F 2 "~" V 7830 4850 30  0000 C CNN
+F 3 "https://www.seielect.com/catalog/SEI-CF_CFM.pdf" H 7900 4850 30  0001 C CNN
+F 4 "Stackpole" H 7900 4850 60  0001 C CNN "MFG Name"
+F 5 "CF14JT22K0" H 7900 4850 60  0001 C CNN "MFG Part Num"
+	1    7900 4850
+	0    -1   -1   0
+$EndComp
 $EndSCHEMATC

Commit message: All Design Files Updated to KiCad v4.0.0_RC1
Parts:
- C1: footprint ~ -> Capacitors_ThroughHole:C_Disc_D6_P5; Characteristics (none) -> CAP CER 10000PF 50V X7R RADIAL; Critical (none) -> N; Description (none) -> 0.1uF MSGEQ7 Bypass Capacitor; MFG Name Vishay -> (none); MFG Part Num K103K15X7RF53L2 -> (none); MFN (none) -> Murata; MFP (none) -> RDER71H104K0M1H03A; Package ID (none) -> PTH_5.00mm; Source (none) -> ANY; Subsystem (none) -> Main
- C2: footprint ~ -> Capacitors_ThroughHole:C_Disc_D6_P5; Characteristics (none) -> CAP CER 10000PF 50V X7R RADIAL; Critical (none) -> N; Description (none) -> 0.1uF Audio DC Decoupling Cap; MFG Name Vishay -> (none); MFG Part Num K103K15X7RF53L2 -> (none); MFN (none) -> Murata; MFP (none) -> RDER71H104K0M1H03A; Package ID (none) -> PTH_5.00mm; Source (none) -> ANY; Subsystem (none) -> Main
- C3: footprint ~ -> Capacitors_ThroughHole:C_Disc_D3_P2.5; Characteristics (none) -> CAP CER 33PF 50V NP0 RADIAL; Critical (none) -> N; Description (none) -> 33pF RC Oscillator Cap; MFG Name Vishay -> (none); MFG Part Num K330J15C0GF5TL2 -> (none); MFN (none) -> Vishay; MFP (none) -> K330J15C0GF5TL2; Package ID (none) -> PTH_2.50mm; Source (none) -> ANY; Subsystem (none) -> Main
- C4: footprint ~ -> Capacitors_ThroughHole:C_Disc_D6_P5; Characteristics (none) -> CAP CER 10000PF 50V X7R RADIAL; Critical (none) -> N; Description (none) -> 0.1uF VSS Capacitor; MFG Name Vishay -> (none); MFG Part Num K103K15X7RF53L2 -> (none); MFN (none) -> Murata; MFP (none) -> RDER71H104K0M1H03A; Package ID (none) -> PTH_5.00mm; Source (none) -> ANY; Subsystem (none) -> Main
- J1: footprint (none) -> Pin_Headers:Pin_Header_Straight_1x05; symbol BREAKOUT_BOARD_HEADER -> Breakout_Board_Header; Characteristics (none) -> CONN HEADER .100\" SNGL STR 5POS; Critical (none) -> N; Description (none) -> .1\" Six Pin Header; MFG Name Sullins Connector -> (none); MFG Part Num PREC040SAAN-RC -> (none); MFN (none) -> Sullins Connector; MFP (none) -> PREC005SAAN-RC; Package ID (none) -> PTH; Source (none) -> ANY; Subsystem (none) -> Main
- J2: footprint (none) -> Project_Footprints:3.5mm_Stereo_Jack_SJ1-3523NG; Critical (none) -> N; Source (none) -> ANY
- R1: footprint ~ -> Project_Footprints:PTH_Resistor; Characteristics (none) -> RES 200K OHM 1/4W 5% CARBON FILM; Critical (none) -> N; Description (none) -> 200K RC Oscillator Resistor; MFG Name Stackpole -> (none); MFG Part Num CF14JT200K -> (none); MFN (none) -> Stackpole; MFP (none) -> CF14JT200K; Package ID (none) -> PTH_Resistor; Source (none) -> ANY; Subsystem (none) -> Main
- R2, R3: footprint ~ -> Project_Footprints:PTH_Resistor; Characteristics (none) -> RES 22K OHM 1/4W 5% CARBON FILM; Critical (none) -> N; Description (none) -> 22K Audio Input Resistor; MFG Name Stackpole -> (none); MFG Part Num CF14JT22K0 -> (none); MFN (none) -> Stackpole; MFP (none) -> CF14JT22K0; Package ID (none) -> PTH_Resistor; Source (none) -> ANY; Subsystem (none) -> Main
- U1: footprint (none) -> Housings_DIP:DIP-8_W7.62mm_LongPads; Characteristics (none) -> Seven Band Graphic Equalizer Display Filter DIP8; Critical (none) -> Y; Description (none) -> Seven Band Graphic Equalizer; MFG Name Mixed Signal Integration -> (none); MFG Part Num MSGEQ7 -> (none); MFN (none) -> Mixed Signal Integration; MFP (none) -> MSGEQ7; Notes (none) -> Must be purchased direct from MFN - Not In Distribution!; Package ID (none) -> PTH_DIP8; Source (none) -> ANY; Subsystem (none) -> Main
Connections:
- wire segments 35 -> 39
